Commit message: added atom
changes since last commit :
- added atom

near term features pending (deadline - 16th June, 2023) :
-

long term features pending :
-

current commit policy - commit to main

File: src/atom/urdf/atom.xacro (robot description, xacro)
@@ -171,5 +171,5 @@
 			<origin xyz="0 0 0" rpy="0 0 0"/>
 			<geometry>
-				<mesh filename="package://fredbots/meshes/hokuyo.dae"/>
+				<mesh filename="package://atom/meshes/hokuyo.dae"/>
 			</geometry>
 		</visual>
@@ -286,4 +286,4 @@
 	</gazebo>
 	<!-- Motor, Camera and Lidar Simulation -->
-	<xacro:include filename="$(find fredbots)/urdf/atom.gazebo" />
+	<xacro:include filename="$(find atom)/urdf/atom.gazebo" />
 </robot>

Commit message: atom fix

File: src/atom/urdf/atom.xacro (robot description, xacro)
@@ -171,5 +171,5 @@
 			<origin xyz="0 0 0" rpy="0 0 0"/>
 			<geometry>
-				<mesh filename="package://atom/meshes/hokuyo.dae"/>
+				<mesh filename="package://fredbots/src/atom/meshes/hokuyo.dae"/>
 			</geometry>
 		</visual>
@@ -286,4 +286,4 @@
 	</gazebo>
 	<!-- Motor, Camera and Lidar Simulation -->
-	<xacro:include filename="$(find atom)/urdf/atom.gazebo" />
+	<xacro:include filename="$(find fredbots)/src/atom/urdf/atom.gazebo" />
 </robot>

Commit message: atom visualisation in rviz + default.rviz mods

File: src/atom/urdf/atom.xacro (robot description, xacro)
@@ -190,5 +190,4 @@
 	    <child link="right_wheel_back" />
 	    <axis xyz="0 1 0" rpy="0 0 0" />
-	    <limit effort="10000" velocity="1000" />
 	    <dynamics damping="1.0" friction="1.0" />
 	</joint>
@@ -199,5 +198,4 @@
 	    <child link="right_wheel_front" />
 	    <axis xyz="0 1 0" rpy="0 0 0" />
-	    <limit effort="10000" velocity="1000" />
 	    <dynamics damping="1.0" friction="1.0" />
 	</joint>
@@ -208,5 +206,4 @@
 	    <child link="left_wheel_back" />
 	    <axis xyz="0 1 0" rpy="0 0 0" />
-	    <limit effort="10000" velocity="1000" />
 	    <dynamics damping="1.0" friction="1.0" />
 	</joint>
@@ -217,5 +214,4 @@
 	    <child link="left_wheel_front" />
 	    <axis xyz="0 1 0" rpy="0 0 0" />
-	    <limit effort="10000" velocity="1000" />
 	    <dynamics damping="1.0" friction="1.0" />
 	</joint>
