Commit message: added all bot desciptions + removed 'atom' refs

File: src/bot_1/atom.xacro (robot description, xacro)
@@ -171,5 +171,5 @@
 			<origin xyz="0 0 0" rpy="0 0 0"/>
 			<geometry>
-				<mesh filename="package://atom/meshes/hokuyo.dae"/>
+				<mesh filename="package://fredbots/src/atom/meshes/hokuyo.dae"/>
 			</geometry>
 		</visual>
@@ -286,4 +286,4 @@
 	</gazebo>
 	<!-- Motor, Camera and Lidar Simulation -->
-	<xacro:include filename="$(find atom)/urdf_test/bot_1/atom.gazebo" />
+	<xacro:include filename="$(find fredbots)/src/bot_1/atom.gazebo" />
 </robot>

File: src/bot_3/atom.xacro (robot description, xacro)
@@ -171,5 +171,5 @@
 			<origin xyz="0 0 0" rpy="0 0 0"/>
 			<geometry>
-				<mesh filename="package://atom/meshes/hokuyo.dae"/>
+				<mesh filename="package://fredbots/src/atom/meshes/hokuyo.dae"/>
 			</geometry>
 		</visual>
@@ -286,4 +286,4 @@
 	</gazebo>
 	<!-- Motor, Camera and Lidar Simulation -->
-	<xacro:include filename="$(find atom)/urdf_test/bot_1/atom.gazebo" />
+	<xacro:include filename="$(find fredbots)/src/bot_3/atom.gazebo" />
 </robot>
