Commit message: single bot spawns fully

File: src/atom/multi_urdf/bot_1/atom.xacro (robot description, xacro)
@@ -1,5 +1,5 @@
 <?xml version='1.0'?>
 <robot name="atom" xmlns:xacro="http://www.ros.org/wiki/xacro">
-	<xacro:property name="robot_name" value="atom" />
+	<xacro:property name="robot_name" value="atom_1" />
 	<xacro:property name="robot_chassis_mass" value="15"/>
 	<xacro:property name="robot_chassis_length" value="0.2"/>

Commit message: changed color of bots

File: src/atom/multi_urdf/bot_1/atom.xacro (robot description, xacro)
@@ -241,5 +241,5 @@
 	<!-- Color of bot -->
 	<gazebo reference="left_wheel_front">
-		<material>Gazebo/Green</material>
+		<material>Gazebo/Black</material>
 		<kp>1000000.0</kp> <!-- kp and kd for rubber -->
 		<kd>100.0</kd>
@@ -250,5 +250,5 @@
 	</gazebo>
 	<gazebo reference="left_wheel_back">
-		<material>Gazebo/Green</material>
+		<material>Gazebo/Black</material>
 		<kp>1000000.0</kp> <!-- kp and kd for rubber -->
 		<kd>100.0</kd>
@@ -259,5 +259,5 @@
 	</gazebo>
 	<gazebo reference="right_wheel_front">
-		<material>Gazebo/Green</material>
+		<material>Gazebo/Black</material>
 		<kp>1000000.0</kp> <!-- kp and kd for rubber -->
 		<kd>100.0</kd>
@@ -268,5 +268,5 @@
 	</gazebo>
 	<gazebo reference="right_wheel_back">
-		<material>Gazebo/Green</material>
+		<material>Gazebo/Black</material>
 		<kp>1000000.0</kp> <!-- kp and kd for rubber -->
 		<kd>100.0</kd>
@@ -277,11 +277,11 @@
 	</gazebo>
 	<!--<gazebo reference="right_wheel">
-		<material>Gazebo/Green</material>
+		<material>Gazebo/Black</material>
 	</gazebo>-->
 	<gazebo reference="camera">
-		<material>Gazebo/Red</material>
+		<material>Gazebo/Grey</material>
 	</gazebo>
 	<gazebo reference="chassis">
-		<material>Gazebo/Blue</material>
+		<material>Gazebo/Green</material>
 	</gazebo>
 	<!-- Motor, Camera and Lidar Simulation -->

File: src/atom/multi_urdf/bot_2/atom.xacro (robot description, xacro)
@@ -241,5 +241,5 @@
 	<!-- Color of bot -->
 	<gazebo reference="left_wheel_front">
-		<material>Gazebo/Green</material>
+		<material>Gazebo/Black</material>
 		<kp>1000000.0</kp> <!-- kp and kd for rubber -->
 		<kd>100.0</kd>
@@ -250,5 +250,5 @@
 	</gazebo>
 	<gazebo reference="left_wheel_back">
-		<material>Gazebo/Green</material>
+		<material>Gazebo/Black</material>
 		<kp>1000000.0</kp> <!-- kp and kd for rubber -->
 		<kd>100.0</kd>
@@ -259,5 +259,5 @@
 	</gazebo>
 	<gazebo reference="right_wheel_front">
-		<material>Gazebo/Green</material>
+		<material>Gazebo/Black</material>
 		<kp>1000000.0</kp> <!-- kp and kd for rubber -->
 		<kd>100.0</kd>
@@ -268,5 +268,5 @@
 	</gazebo>
 	<gazebo reference="right_wheel_back">
-		<material>Gazebo/Green</material>
+		<material>Gazebo/Black</material>
 		<kp>1000000.0</kp> <!-- kp and kd for rubber -->
 		<kd>100.0</kd>
@@ -280,5 +280,5 @@
 	</gazebo>-->
 	<gazebo reference="camera">
-		<material>Gazebo/Red</material>
+		<material>Gazebo/Grey</material>
 	</gazebo>
 	<gazebo reference="chassis">

File: src/atom/multi_urdf/bot_3/atom.xacro (robot description, xacro)
@@ -241,5 +241,5 @@
 	<!-- Color of bot -->
 	<gazebo reference="left_wheel_front">
-		<material>Gazebo/Green</material>
+		<material>Gazebo/Black</material>
 		<kp>1000000.0</kp> <!-- kp and kd for rubber -->
 		<kd>100.0</kd>
@@ -250,5 +250,5 @@
 	</gazebo>
 	<gazebo reference="left_wheel_back">
-		<material>Gazebo/Green</material>
+		<material>Gazebo/Black</material>
 		<kp>1000000.0</kp> <!-- kp and kd for rubber -->
 		<kd>100.0</kd>
@@ -259,5 +259,5 @@
 	</gazebo>
 	<gazebo reference="right_wheel_front">
-		<material>Gazebo/Green</material>
+		<material>Gazebo/Black</material>
 		<kp>1000000.0</kp> <!-- kp and kd for rubber -->
 		<kd>100.0</kd>
@@ -268,5 +268,5 @@
 	</gazebo>
 	<gazebo reference="right_wheel_back">
-		<material>Gazebo/Green</material>
+		<material>Gazebo/Black</material>
 		<kp>1000000.0</kp> <!-- kp and kd for rubber -->
 		<kd>100.0</kd>
@@ -280,8 +280,8 @@
 	</gazebo>-->
 	<gazebo reference="camera">
-		<material>Gazebo/Red</material>
+		<material>Gazebo/Grey</material>
 	</gazebo>
 	<gazebo reference="chassis">
-		<material>Gazebo/Blue</material>
+		<material>Gazebo/Orange</material>
 	</gazebo>
 	<!-- Motor, Camera and Lidar Simulation -->

File: src/atom/multi_urdf/bot_4/atom.xacro (robot description, xacro)
@@ -241,5 +241,5 @@
 	<!-- Color of bot -->
 	<gazebo reference="left_wheel_front">
-		<material>Gazebo/Green</material>
+		<material>Gazebo/Black</material>
 		<kp>1000000.0</kp> <!-- kp and kd for rubber -->
 		<kd>100.0</kd>
@@ -250,5 +250,5 @@
 	</gazebo>
 	<gazebo reference="left_wheel_back">
-		<material>Gazebo/Green</material>
+		<material>Gazebo/Black</material>
 		<kp>1000000.0</kp> <!-- kp and kd for rubber -->
 		<kd>100.0</kd>
@@ -259,5 +259,5 @@
 	</gazebo>
 	<gazebo reference="right_wheel_front">
-		<material>Gazebo/Green</material>
+		<material>Gazebo/Black</material>
 		<kp>1000000.0</kp> <!-- kp and kd for rubber -->
 		<kd>100.0</kd>
@@ -268,5 +268,5 @@
 	</gazebo>
 	<gazebo reference="right_wheel_back">
-		<material>Gazebo/Green</material>
+		<material>Gazebo/Black</material>
 		<kp>1000000.0</kp> <!-- kp and kd for rubber -->
 		<kd>100.0</kd>
@@ -280,8 +280,8 @@
 	</gazebo>-->
 	<gazebo reference="camera">
-		<material>Gazebo/Red</material>
+		<material>Gazebo/Grey</material>
 	</gazebo>
 	<gazebo reference="chassis">
-		<material>Gazebo/Blue</material>
+		<material>Gazebo/Yellow</material>
 	</gazebo>
 	<!-- Motor, Camera and Lidar Simulation -->

Commit message: fixed bot similarity error

File: src/atom/multi_urdf/bot_1/atom.xacro (robot description, xacro)
@@ -283,7 +283,7 @@
 	</gazebo>
 	<gazebo reference="chassis">
-		<material>Gazebo/Yellow</material>
+		<material>Gazebo/Red</material>
 	</gazebo>
 	<!-- Motor, Camera and Lidar Simulation -->
-	<xacro:include filename="$(find fredbots)/src/atom/multi_urdf/bot_2/atom.gazebo" />
+	<xacro:include filename="$(find fredbots)/src/atom/multi_urdf/bot_1/atom.gazebo" />
 </robot>
