Commit message: color change

File: src/atom/multi_urdf/bot_2/atom.xacro (robot description, xacro)
@@ -283,5 +283,5 @@
 	</gazebo>
 	<gazebo reference="chassis">
-		<material>Gazebo/Blue</material>
+		<material>Gazebo/Yellow</material>
 	</gazebo>
 	<!-- Motor, Camera and Lidar Simulation -->

File: src/atom/multi_urdf/bot_3/atom.xacro (robot description, xacro)
@@ -283,5 +283,5 @@
 	</gazebo>
 	<gazebo reference="chassis">
-		<material>Gazebo/Blue</material>
+		<material>Gazebo/Orange</material>
 	</gazebo>
 	<!-- Motor, Camera and Lidar Simulation -->

File: src/atom/multi_urdf/bot_4/atom.xacro (robot description, xacro)
@@ -283,5 +283,5 @@
 	</gazebo>
 	<gazebo reference="chassis">
-		<material>Gazebo/Blue</material>
+		<material>Gazebo/Red</material>
 	</gazebo>
 	<!-- Motor, Camera and Lidar Simulation -->

Commit message: single bot spawns fully in rviz

File: src/atom/multi_urdf/bot_2/atom.xacro (robot description, xacro)
@@ -1,5 +1,5 @@
 <?xml version='1.0'?>
 <robot name="atom" xmlns:xacro="http://www.ros.org/wiki/xacro">
-	<xacro:property name="robot_name" value="atom" />
+	<xacro:property name="robot_name" value="atom_2" />
 	<xacro:property name="robot_chassis_mass" value="15"/>
 	<xacro:property name="robot_chassis_length" value="0.2"/>

Commit message: Bot colors and bot IDs which can input colors.

File: src/atom/multi_urdf/bot_2/atom.xacro (robot description, xacro)
@@ -283,5 +283,5 @@
 	</gazebo>
 	<gazebo reference="chassis">
-		<material>Gazebo/Yellow</material>
+		<material>Gazebo/Orange</material>
 	</gazebo>
 	<!-- Motor, Camera and Lidar Simulation -->

File: src/atom/multi_urdf/bot_3/atom.xacro (robot description, xacro)
@@ -283,5 +283,5 @@
 	</gazebo>
 	<gazebo reference="chassis">
-		<material>Gazebo/Orange</material>
+		<material>Gazebo/Green</material>
 	</gazebo>
 	<!-- Motor, Camera and Lidar Simulation -->
